File: ESPgarage.kicad_sch (KiCad schematic)
At the start: 1 part

Commit message: Add
Parts:
- added D1: B240, Diode_SMD:D_SMB, symbol Diode:B240
- added U1: MAX5035BUSA, Package_SO:SOIC-8_3.9x4.9mm_P1.27mm, symbol Regulator_Switching:MAX5035BUSA
- gave numbers to parts that had none: 1
Connections:
- new net: D1.1 (K), U1.1 (BST)
- new net GND: D1.2 (A)
Changed lines of the file:
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@@
 (kicad_sch (version 20211123) (generator eeschema)
   (paper "A4")
+  (wire (pts (xy 60.96 50.8) (xy 76.2 50.8))
+    (stroke (width 0) (type default) (color 0 0 0 0))
+  )
+  (wire (pts (xy 76.2 59.69) (xy 76.2 62.23))
+    (stroke (width 0) (type default) (color 0 0 0 0))
+  )
+  (wire (pts (xy 76.2 50.8) (xy 76.2 52.07))
+    (stroke (width 0) (type default) (color 0 0 0 0))
+  )
   (symbol (lib_id "Device:R_US") (at 124.46 87.63 0) (unit 1)
     (in_bom yes) (on_board yes) (fields_autoplaced)
-    (property "Reference" "R?" (id 0) (at 127 86.3599 0)
+    (property "Reference" "R1" (id 0) (at 127 86.3599 0)
       (effects (font (size 1.27 1.27)) (justify left))
     )
@@
     (pin "2")
   )
+  (symbol (lib_id "Regulator_Switching:MAX5035BUSA") (at 50.8 55.88 0) (unit 1)
+    (in_bom yes) (on_board yes) (fields_autoplaced)
+    (property "Reference" "U1" (id 0) (at 50.8 43.18 0))
+    (property "Value" "MAX5035BUSA" (id 1) (at 50.8 45.72 0))
+    (property "Footprint" "Package_SO:SOIC-8_3.9x4.9mm_P1.27mm" (id 2) (at 54.61 64.77 0)
+      (effects (font (size 1.27 1.27) italic) (justify left) hide)
+    )
+    (property "Datasheet" "http://datasheets.maximintegrated.com/en/ds/MAX5035.pdf" (id 3) (at 50.8 57.15 0)
+      (effects (font (size 1.27 1.27)) hide)
+    )
+    (pin "1")
+    (pin "2")
+    (pin "3")
+    (pin "4")
+    (pin "5")
+    (pin "6")
+    (pin "7")
+    (pin "8")
+  )
+  (symbol (lib_id "power:GND") (at 76.2 62.23 0) (unit 1)
+    (in_bom yes) (on_board yes)
+    (property "Reference" "#PWR0101" (id 0) (at 76.2 68.58 0)
+      (effects (font (size 1.27 1.27)) hide)
+    )
+    (property "Value" "GND" (id 1) (at 76.2 67.31 0))
+    (property "Footprint" "" (id 2) (at 76.2 62.23 0)
+      (effects (font (size 1.27 1.27)) hide)
+    )
+    (property "Datasheet" "" (id 3) (at 76.2 62.23 0)
+      (effects (font (size 1.27 1.27)) hide)
+    )
+    (pin "1")
+  )
+  (symbol (lib_id "Diode:B240") (at 76.2 55.88 270) (unit 1)
+    (in_bom yes) (on_board yes) (fields_autoplaced)
+    (property "Reference" "D1" (id 0) (at 78.74 54.2924 90)
+      (effects (font (size 1.27 1.27)) (justify left))
+    )
+    (property "Value" "B240" (id 1) (at 78.74 56.8324 90)
+      (effects (font (size 1.27 1.27)) (justify left))
+    )
+    (property "Footprint" "Diode_SMD:D_SMB" (id 2) (at 71.755 55.88 0)
+      (effects (font (size 1.27 1.27)) hide)
+    )
+    (property "Datasheet" "http://www.jameco.com/Jameco/Products/ProdDS/1538777.pdf" (id 3) (at 76.2 55.88 0)
+      (effects (font (size 1.27 1.27)) hide)
+    )
+    (pin "1")
+    (pin "2")
+  )
   (sheet_instances
     (path "/" (page "1"))
   )
   (symbol_instances
+    (path "/bcb47aa9-51d2-412b-9924-7bda545dd7c1"
+      (reference "#PWR0101") (unit 1) (value "GND") (footprint "")
+    )
+    (path "/e5fa8627-e279-4dc9-a162-8ee6d8aa13b0"
+      (reference "D1") (unit 1) (value "B240") (footprint "Diode_SMD:D_SMB")
+    )
     (path "/759788bd-3cb9-4d38-b58c-5cb10b7dca6b"
-      (reference "R?") (unit 1) (value "R_US") (footprint "")
+      (reference "R1") (unit 1) (value "R_US") (footprint "")
+    )
+    (path "/a90361cd-254c-4d27-ae1f-9a6c85bafe28"
+      (reference "U1") (unit 1) (value "MAX5035BUSA") (footprint "Package_SO:SOIC-8_3.9x4.9mm_P1.27mm")
     )
   )
